Commit message: human-slim

File: gazebo_models/humanoid/humanoid-fat.urdf (robot description, URDF)
Before this commit: robot humanoid, 10 links, 9 joints
Links:
- link Head_link: geometry collision box size=0.15 0.15 0.2; visual box size=0.15 0.15 0.2
- link LeftLeg_link: geometry collision cylinder length=0.7 radius=0.05; visual cylinder length=0.7 radius=0.05
- link RightLeg_link: geometry collision cylinder length=0.7 radius=0.05; visual cylinder length=0.7 radius=0.05
- link Torso_link: geometry collision box size=0.15 0.3 0.6; visual box size=0.15 0.3 0.6
Joints:
- joint Head_joint: origin xyz=0.0 0.0 1.38 rpy=0.0 0.0 0.0 -> xyz=0.0 0.0 1.4 rpy=0.0 0.0 0.0
- joint LeftFoot_joint: origin xyz=0.0 0.01 -0.7 rpy=0.0 0.0 0.0 -> xyz=0.0 0.0 -0.7 rpy=0.0 0.0 0.0
- joint LeftLeg_joint: origin xyz=0.0 0.05 0.8 rpy=0.0 0.0 0.0 -> xyz=0.0 0.1 0.8 rpy=0.0 0.0 0.0
- joint LeftUpperArm_joint: origin xyz=0.0 0.1 1.3 rpy=0.0 0.0 0.0 -> xyz=0.0 0.15 1.3 rpy=0.0 0.0 0.0
- joint RightFoot_joint: origin xyz=0.0 -0.01 -0.7 rpy=0.0 0.0 0.0 -> xyz=0.0 0.0 -0.7 rpy=0.0 0.0 0.0
- joint RightLeg_joint: origin xyz=0.0 -0.05 0.8 rpy=0.0 0.0 0.0 -> xyz=0.0 -0.1 0.8 rpy=0.0 0.0 0.0
- joint RightUpperArm_joint: origin xyz=0.0 -0.1 1.3 rpy=0.0 0.0 0.0 -> xyz=0.0 -0.15 1.3 rpy=0.0 0.0 0.0
