Commit message: target:humanoid

File: gazebo_models/humanoid/humanoid.urdf (robot description, URDF)
Before this commit: robot humanoid, 8 links, 7 joints
Joints:
- joint LeftForeArm_joint: limit lower=-0.7854 upper=0.7854 effort=30 velocity=1.0 -> lower=-0.0 upper=0.0 effort=30 velocity=1.0
- joint RightForeArm_joint: limit lower=-0.7854 upper=0.7854 effort=30 velocity=1.0 -> lower=-0.0 upper=0.0 effort=30 velocity=1.0

Commit message: targetline change

File: gazebo_models/humanoid/humanoid.urdf (robot description, URDF)
Before this commit: robot humanoid, 8 links, 7 joints
Links:
- removed link Leftleg_link
- removed link Rightleg_link
- added link LeftFoot_link, mass 50; collision box size=0.3 0.15 0.1; visual box size=0.3 0.15 0.1
- added link LeftLeg_link, mass 10; collision cylinder length=0.7 radius=0.05; visual cylinder length=0.7 radius=0.05
- added link RightFoot_link, mass 50; collision box size=0.3 0.15 0.1; visual box size=0.3 0.15 0.1
- added link RightLeg_link, mass 10; collision cylinder length=0.7 radius=0.05; visual cylinder length=0.7 radius=0.05
Joints:
- removed joint Leftleg_joint
- removed joint Rightleg_joint
- added joint LeftFoot_joint: type fixed, parent LeftLeg_link, child LeftFoot_link, origin xyz=0.0 0.0 -0.7 rpy=0.0 0.0 0.0, axis 0 0 1
- added joint LeftLeg_joint: type revolute, parent Torso_link, child LeftLeg_link, origin xyz=0.0 0.1 0.8 rpy=0.0 0.0 0.0, axis 1 0 0, limit lower=-0.5 upper=0.5 effort=30 velocity=1.0
- added joint RightFoot_joint: type fixed, parent RightLeg_link, child RightFoot_link, origin xyz=0.0 0.0 -0.7 rpy=0.0 0.0 0.0, axis 0 0 1
- added joint RightLeg_joint: type revolute, parent Torso_link, child RightLeg_link, origin xyz=0.0 -0.1 0.8 rpy=0.0 0.0 0.0, axis 1 0 0, limit lower=-0.5 upper=0.5 effort=30 velocity=1.0

Commit message: moving leg

File: gazebo_models/humanoid/humanoid.urdf (robot description, URDF)
Before this commit: robot humanoid, 10 links, 9 joints
Links:
- link LeftFoot_link: mass 50 -> 100
- link RightFoot_link: mass 50 -> 100
- link Torso_link: mass 1 -> 10
Joints:
- joint LeftLeg_joint: axis 1 0 0 -> 0 0 1; limit lower=-0.5 upper=0.5 effort=30 velocity=1.0 -> lower=-0.3 upper=0.3 effort=30000 velocity=100.0; type revolute -> prismatic
- joint RightLeg_joint: axis 1 0 0 -> 0 0 1; limit lower=-0.5 upper=0.5 effort=30 velocity=1.0 -> lower=-0.3 upper=0.3 effort=30000 velocity=100.0; mimic (none) -> joint=LeftLeg_joint multiplier=1 offset=0; type revolute -> prismatic

Commit message: new humanoid, new targetline

File: gazebo_models/humanoid/humanoid.urdf (robot description, URDF)
Before this commit: robot humanoid, 10 links, 9 joints
Joints:
- joint Head_joint: origin xyz=0.0 0.0 1.38 rpy=0.0 0.0 0.0 -> xyz=0.0 0.0 1.4 rpy=0.0 0.0 0.0
