Commit message: test

File: gazebo_models/humanoid/humanoid-slim.urdf (robot description, URDF)
Before this commit: robot humanoid, 10 links, 9 joints
Joints:
- joint LeftForeArm_joint: limit lower=-0.0 upper=0.0 effort=30 velocity=1.0 -> lower=-0.5 upper=0.5 effort=30000 velocity=10000.0
- joint RightForeArm_joint: limit lower=-0.0 upper=0.0 effort=30 velocity=1.0 -> lower=-0.5 upper=0.5 effort=30000 velocity=10000.0

File: gazebo_models/humanoid/humanoid-stout.urdf (robot description, URDF)
Before this commit: robot humanoid, 10 links, 9 joints
Joints:
- joint LeftForeArm_joint: limit lower=-0.0 upper=0.0 effort=30 velocity=1.0 -> lower=-0.5 upper=0.5 effort=30000 velocity=1000.0
- joint RightForeArm_joint: limit lower=-0.0 upper=0.0 effort=30 velocity=1.0 -> lower=-0.5 upper=0.5 effort=30000 velocity=1000.0
