Commit message: humanoid_pose

File: gazebo_models/humanoid/humanoid-static-left.urdf (robot description, URDF)
Before this commit: robot humanoid, 10 links, 9 joints
Links:
- link LeftForeArm_link: geometry 
- link LeftUpperArm_link: geometry 

File: gazebo_models/humanoid/humanoid-static-right.urdf (robot description, URDF)
Before this commit: robot humanoid, 10 links, 9 joints
Links:
- link RightForeArm_link: geometry 
- link RightUpperArm_link: geometry 
